Commit message: Respostas do exercicio 4

File: week-2/.ipynb_checkpoints/arm_3r-checkpoint.urdf (robot description, URDF)
Before this commit: robot pend_robot, 7 links, 6 joints
Joints:
- removed joint first_joint
- added joint base_joint: type continuous, parent base_link, child body_link, origin xyz=0 0 0 rpy=0 0 0, axis 0 0 1
